File: src/pcb/form-neo/form-neo.kicad_pcb (KiCad board)
At the start: 2 copper layers, 282.5 x 128.4 mm, 123 parts, among them SW1 SW_Push, SW10 SW_Push, SW11 SW_Push, SW12 SW_Push, SW13 SW_Push, SW14 SW_Push, SW15 SW_Push, SW16 SW_Push, SW17 SW_Push, SW18 SW_Push, SW19 SW_Push, SW2 SW_Push, SW20 SW_Push, SW21 SW_Push, SW22 SW_Push, SW23 SW_Push, SW24 SW_Push, SW25 SW_Push, SW26 SW_Push, SW27 SW_Push, SW28 SW_Push, SW29 SW_Push, SW3 SW_Push, SW30 SW_Push, SW31 SW_Push, SW32 SW_Push, SW33 SW_Push, SW34 SW_Push, SW35 SW_Push, SW36 SW_Push, SW37 SW_Push, SW38 SW_Push, SW39 SW_Push, SW4 SW_Push, SW40 SW_Push, SW41 SW_Push, SW42 SW_Push, SW43 SW_Push, SW44 SW_Push, SW45 SW_Push, SW46 SW_Push, SW47 SW_Push, SW48 SW_Push, SW49 SW_Push, SW5 SW_Push, SW50 SW_Push, SW51 SW_Push, SW52 SW_Push, SW53 SW_Push, SW54 SW_Push, SW55 SW_Push, SW56 SW_Push, SW57 SW_Push, SW58 SW_Push, SW59 SW_Push, SW6 SW_Push, SW60 SW_Push, SW61 SW_Push, SW62 SW_Push, SW7 SW_Push, SW8 SW_Push, SW9 SW_Push, U1 rp2040-zero

Commit message: Set revision
Parts:
- moved D18 45.2 mm to (171.3, 68.0)
- moved D19 45.2 mm to (218.0, 70.9)
- moved D20 45.2 mm to (236.3, 65.2)
- moved D30 45.2 mm to (168.0, 86.8)
- moved D33 45.2 mm to (258.0, 78.3)
- moved D34 45.2 mm to (277.2, 77.4)
- moved D36 45.2 mm to (315.5, 75.4)
- moved D42 45.2 mm to (164.6, 105.5)
- moved D43 45.2 mm to (224.6, 108.4)
- moved D45 45.2 mm to (261.3, 97.1)
- moved D47 45.2 mm to (300.1, 97.5)
- moved D52 45.2 mm to (150.2, 124.7)
- moved D53 45.2 mm to (155.5, 126.4)
- moved D60 45.2 mm to (322.1, 113.0)
- moved SW20 45.2 mm to (245.0, 66.6)
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Other:
- board text added: "${TITLE}"
- board text added: "rev${REVISION}"
